File: hardware/opod.kicad_pcb (KiCad board)
At the start: 2 copper layers, 1 part, among them U1 STM32F411CEUx

Commit message: Hello, World x2
Parts:
- added U2: MTCH6102, Package_DFN_QFN:UQFN-28-1EP_4x4mm_P0.4mm_EP2.35x2.35mm, F.Cu at (165.3, 104.8)
- added U3: W25Q128JVP, Package_SON:WSON-8-1EP_6x5mm_P1.27mm_EP3.4x4.3mm, F.Cu at (150.2, 106.8)
- U1: value STM32F411CEUx -> RP2350A; footprint Package_DFN_QFN:QFN-48-1EP_7x7mm_P0.5mm_EP5.6x5.6mm -> Package_DFN_QFN:QFN-60-1EP_7x7mm_P0.4mm_EP3.4x3.4mm
- moved U1 25.9 mm to (156.4, 97.3)
Connections:
- U1 pad 1: unconnected-(U1-VBAT-Pad1) -> Net-(U1-IOVDD-Pad1)
- U1 pad 11: unconnected-(U1-PA1-Pad11) -> Net-(U1-IOVDD-Pad1)
- U1 pad 20: unconnected-(U1-PB2-Pad20) -> Net-(U1-IOVDD-Pad1)
- U1 pad 23: Net-(U1-VSS-Pad23) -> Net-(U1-DVDD-Pad23)
- U1 pad 30: unconnected-(U1-PA9-Pad30) -> Net-(U1-IOVDD-Pad1)
- U1 pad 35: Net-(U1-VSS-Pad23) -> unconnected-(U1-GPIO23-Pad35)
- U1 pad 38: unconnected-(U1-PA15-Pad38) -> Net-(U1-IOVDD-Pad1)
- U1 pad 39: unconnected-(U1-PB3-Pad39) -> Net-(U1-DVDD-Pad23)
- U1 pad 45: unconnected-(U1-PB8-Pad45) -> Net-(U1-IOVDD-Pad1)
- U1 pad 47: Net-(U1-VSS-Pad23) -> unconnected-(U1-VREG_PGND-Pad47)
- U1 pad 49: Net-(U1-VSS-Pad23) -> unconnected-(U1-VREG_VIN-Pad49)
- U1 pad 6: unconnected-(U1-PH1-Pad6) -> Net-(U1-DVDD-Pad23)

Commit message: wiring stuff
Parts:
- added C1: 4.7u, Capacitor_SMD:C_0402_1005Metric, F.Cu at (161.3, 110.4)
- added C10: 1u, Capacitor_SMD:C_0402_1005Metric, F.Cu at (164.2, 118.3)
- added C2: 1u, Capacitor_SMD:C_0402_1005Metric, F.Cu at (161.3, 112.4)
- added C3: 4.7u, Capacitor_SMD:C_0402_1005Metric, F.Cu at (161.3, 114.3)
- added C4: 1u, Capacitor_SMD:C_0402_1005Metric, F.Cu at (161.3, 116.3)
- added C5: 1u, Capacitor_SMD:C_0402_1005Metric, F.Cu at (161.3, 118.3)
- added C6: 1u, Capacitor_SMD:C_0402_1005Metric, F.Cu at (164.2, 110.4)
- added C7: 1u, Capacitor_SMD:C_0402_1005Metric, F.Cu at (164.2, 112.4)
- added C8: 1u, Capacitor_SMD:C_0402_1005Metric, F.Cu at (164.2, 114.3)
- added C9: 1u, Capacitor_SMD:C_0402_1005Metric, F.Cu at (164.2, 116.3)
- added D1: MBR0530, Diode_SMD:D_SOD-123, F.Cu at (186.7, 105.6)
- added D2: MBR0530, Diode_SMD:D_SOD-123, F.Cu at (184.9, 109.2)
- added D3: MBR0530, Diode_SMD:D_SOD-123, F.Cu at (185.2, 112.6)
- added J1: USB_C_Receptacle_USB2.0_16P, Connector_USB:USB_C_Receptacle_XKB_U262-16XN-4BVC11, F.Cu at (165.7, 102.7)
- added J2: Conn_01x24_Pin, Connector_FFC-FPC:Hirose_FH12-24S-0.5SH_1x24-1MP_P0.50mm_Horizontal, F.Cu at (191.9, 98.8)
- added JP1: Jumper_2_Bridged, Jumper:SolderJumper-2_P1.3mm_Bridged_Pad1.0x1.5mm, F.Cu at (169.7, 111.2)
- added Q1: Si1308EDL, Package_TO_SOT_SMD:SOT-323_SC-70, F.Cu at (190.0, 105.9)
- added R1: 2.2, Resistor_SMD:R_0402_1005Metric, F.Cu at (167.1, 113.9)
- added R2: 1M, Resistor_SMD:R_0402_1005Metric, F.Cu at (167.1, 115.9)
- added TP1: TestPoint, TestPoint:TestPoint_Pad_D1.5mm, F.Cu at (167.4, 118.7)
- added U4: TLV320DAC3101, Package_DFN_QFN:QFN-32-1EP_5x5mm_P0.5mm_EP3.45x3.45mm, F.Cu at (207.5, 98.9)
- added U5: BQ25895RTW, Package_DFN_QFN:Texas_RTW_WQFN-24-1EP_4x4mm_P0.5mm_EP2.7x2.7mm, F.Cu at (148.7, 101.1)
- moved U3 49.6 mm to (198.1, 119.6)
- moved U2 41.7 mm to (206.9, 107.7)
- moved U1 38.9 mm to (187.3, 120.9)
Connections:
- U2 pad 1: unconnected-(U2-RX11-Pad1) -> Net-(J3-Pin_12)
- U2 pad 10: unconnected-(U2-RX14-Pad10) -> Net-(J3-Pin_15)
- U2 pad 13: unconnected-(U2-RXO-Pad13) -> Net-(J3-Pin_1)
- U2 pad 14: unconnected-(U2-RX1-Pad14) -> Net-(J3-Pin_2)
- U2 pad 15: unconnected-(U2-RX2-Pad15) -> Net-(J3-Pin_3)
- U2 pad 18: unconnected-(U2-RX3-Pad18) -> Net-(J3-Pin_4)
- U2 pad 19: unconnected-(U2-RX4-Pad19) -> Net-(J3-Pin_5)
- U2 pad 2: unconnected-(U2-RX12-Pad2) -> Net-(J3-Pin_13)
- U2 pad 20: unconnected-(U2-RX5-Pad20) -> Net-(J3-Pin_6)
- U2 pad 21: unconnected-(U2-RX6-Pad21) -> Net-(J3-Pin_7)
- U2 pad 22: unconnected-(U2-RX7-Pad22) -> Net-(J3-Pin_8)
- U2 pad 23: unconnected-(U2-RX8-Pad23) -> Net-(J3-Pin_9)
- U2 pad 27: unconnected-(U2-RX9-Pad27) -> Net-(J3-Pin_10)
- U2 pad 28: unconnected-(U2-RX10-Pad28) -> Net-(J3-Pin_11)
- U2 pad 4: unconnected-(U2-RX13-Pad4) -> Net-(J3-Pin_14)
