File: hardware/audio.kicad_sch (KiCad schematic)
At the start: 1 part, among them U4 TLV320DAC3101

Commit message: charging circuit
Connections:
- no-connect marks 0 -> 2
Changed lines of the file:
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@@
 	(generator_version "10.0")
 	(paper "A4")
+	(no_connect
+		(at 111.76 91.44)
+	)
+	(no_connect
+		(at 111.76 93.98)
+	)
 	(symbol
 		(lib_id "Analog_DAC:TLV320DAC3101")
