File: hardware/charging.kicad_sch (KiCad schematic)
At the start: 6 parts, among them U5 BQ25895RTW

Commit message: charging circuit
Parts:
- added C17: 4.7u, symbol Device:C
- added C18: 47n, symbol Device:C_Small
- added C19, C20, C23, C24, C25, C27: 10u, symbol Device:C
- added C21, C28, C30: 1u, symbol Device:C
- added C22, C26, C29, C31: 100n, symbol Device:C
- added D4: LED, symbol Device:LED
- added L2: 2.2u, symbol Device:L
- added R10, R12, R8, R9: 5.1k, symbol Device:R_Small
- added R11: 260R, symbol Device:R_Small
- added R13, R14: 10k, symbol Device:R_Small
- added R15: 1k, symbol Device:R_Small
- added SW1: SW_Push_45deg, symbol Switch:SW_Push_45deg
- added U7: TLV76733DRVx, Package_SON:WSON-6-1EP_2x2mm_P0.65mm_EP1x1.6mm_ThermalVias, symbol Regulator_Linear:TLV76733DRVx
Connections:
- net GND: now also U5.9 (~{CE}), C17.2, C19.2, C20.2, C21.2, C22.2, C23.2, C24.2, C25.2, C26.2, C27.2, C28.2, C29.2, C30.2, C31.2, R11.2, R13.2, SW1.1, U7.3 (GND), U7.5 (GND), U7.7 (PAD)
- net at U5.10 (ILIM): now also R11.1
- net at U5.11 (TS): now also R12.2, R13.1
- net at U5.12 (~{QON}): now also SW1.2
- net VSYS: now reaches U5.15 (SYS), U5.16 (SYS)
- net VSYS: now also C19.1, C20.1, C21.1, C22.1, C28.1, C29.1, L2.2, R14.1, R15.2, U7.4 (EN), U7.6 (IN)
- net at U5.19 (SW), U5.20 (SW): now also C18.1, L2.1
- net at U5.21 (BTST): now also C18.2
- net at U5.22 (REGN): now also C17.1, R12.1
- net PMID: now reaches U5.23 (PMID)
- net PMID: now also C23.1, C24.1, C25.1, C26.1, C27.1
- net CHG_SCL: now reaches U5.5 (SCL)
- net CHG_SCL: now also R8.2
- net CHG_SDA: now reaches U5.6 (SDA)
- net CHG_SDA: now also R9.2
- net CHG_INT: now reaches U5.7 (~{INT})
- net CHG_INT: now also R10.2
- net CHG_OTG: now reaches U5.8 (OTG)
- net STAT: no longer names the net of U5.4 (STAT)
- net STAT: now also D4.2 (A), R14.2
- new net: D4.1 (K), R15.1
- new net +3V3: C30.1, C31.1, R10.1, R8.1, R9.1, U7.1 (OUT), U7.2 (SNS)
Other:
- moved on the sheet: BT1, C11, C12, C13, C14, U5
