File: hardware/storage.kicad_sch (KiCad schematic)
At the start: 2 parts, among them J4 Micro_SD_Card, U3 W25Q128JVP

Commit message: charging circuit
Parts:
- added C32, C33: 100n, symbol Device:C
Connections:
- net +3V3: now also J4.4 (VDD), C32.1, C33.1
- net GND: now also J4.6 (VSS), C32.2, C33.2
